File: Voicemeeter/_saved_file5AF6330C.sch (KiCad schematic (older format))
At the start: 10 parts, among them U401 74HC4051, U402 74HC4051, U403 74HC4051, U404 74HC4051, U405 74HC4051, U406 74HC4051, U407 74HC4051, U408 74HC4051, U409 74HC4051, U410 74HC4051

Commit message: fsd
Connections:
- net DA12: now also U403.12 (X3); no longer U403.14 (X1)
- net DA13: now also U403.13 (X0); no longer U403.15 (X2)
- net DA14: now also U403.14 (X1); no longer U403.12 (X3)
- net DA22: now also U403.15 (X2); no longer U403.5 (X5)
- net DA23: now also U403.1 (X4); no longer U403.13 (X0)
- net DA24: now also U403.2 (X6); no longer U403.1 (X4)
- net HA11: now also U401.15 (X2); no longer U401.13 (X0)
- net HA12: now also U401.2 (X6); no longer U401.14 (X1)
- net HA13: now also U401.1 (X4); no longer U401.15 (X2)
- net HA21: now also U401.4 (X7); no longer U401.12 (X3)
- net HA22: now also U401.5 (X5); no longer U401.1 (X4)
- net HA23: now also U401.14 (X1); no longer U401.5 (X5)
- net HA31: now also U401.13 (X0); no longer U401.2 (X6)
- net HA32: now also U401.12 (X3); no longer U401.4 (X7)
- net HA33: now also U403.5 (X5); no longer U403.2 (X6)
- net OD52: now also U410.5 (X5); no longer U410.4 (X7)
- net OD53: now also U410.4 (X7); no longer U410.5 (X5)
- net M01 renamed M1
- net M02 renamed M2
- net M03 renamed M3
