File: Voicemeeter/_saved_test.sch (KiCad schematic (older format))
At the start: 0 parts

Commit message: fsd
Changed lines of the file:
@@
 F3 "OA[1..5]" I L 4000 3150 60
 F4 "DA[11..24]" I L 4000 3250 60
-F5 "M[01..27]" O R 5450 2950 60
+F5 "M[1..27]" O R 5450 2950 60
 F6 "HD[11..38]" I L 4000 2850 60
 F7 "DD[11..28]" I L 4000 2950 60
@@
 F0 "STM" 60
 F1 "file5AE700A4.sch" 60
-F2 "M[01..27]" I L 6250 2950 60
+F2 "M[1..27]" I L 6250 2950 60
 F3 "SK[1..2]" O R 7750 2950 60
 $EndSheet
