File: Voicemeeter/file5AE49270.sch (KiCad schematic (older format))
At the start: 132 parts, among them SW201 SW_SPDT, SW202 SW_SPDT, SW203 SW_SPDT, SW204 SW_SPDT, SW205 SW_SPDT, SW206 SW_SPDT, SW207 SW_SPDT, SW208 SW_SPDT, SW209 SW_SPDT, SW210 SW_SPDT, SW211 SW_SPDT, SW212 SW_SPDT, SW213 SW_SPDT, SW214 SW_SPDT, SW215 SW_SPDT, SW216 SW_SPDT, SW217 SW_SPDT, SW218 SW_SPDT, SW219 SW_SPDT, SW220 SW_SPDT, SW221 SW_SPDT, SW222 SW_SPDT, SW223 SW_SPDT, SW224 SW_SPDT, SW225 SW_SPDT, SW226 SW_SPDT, SW227 SW_SPDT, SW228 SW_SPDT, SW229 SW_SPDT, SW230 SW_SPDT, SW231 SW_SPDT, SW232 SW_SPDT, SW233 SW_SPDT, SW234 SW_SPDT, SW235 SW_SPDT, SW236 SW_SPDT, SW237 SW_SPDT, SW238 SW_SPDT, SW239 SW_SPDT, SW240 SW_SPDT, SW241 SW_SPDT, SW242 SW_SPDT, SW243 SW_SPDT, SW244 SW_SPDT, SW245 SW_SPDT, SW246 SW_SPDT, SW247 SW_SPDT, SW248 SW_SPDT, SW249 SW_SPDT, SW250 SW_SPDT, SW251 SW_SPDT, SW252 SW_SPDT, SW253 SW_SPDT, SW254 SW_SPDT, SW255 SW_SPDT

Commit message: asf
Parts:
- removed SW201, SW202, SW203, SW204, SW205, SW206, SW207, SW208, SW209, SW210, SW211, SW212, SW213, SW214, SW215, SW216, SW217, SW218, SW219, SW220, SW221, SW222, SW223, SW224, SW225, SW226, SW227, SW228, SW229, SW230, SW231, SW232, SW233, SW234, SW235, SW236, SW237, SW238, SW239, SW240, SW241, SW242, SW243, SW244, SW245, SW246, SW247, SW248, SW249, SW250, SW251, SW252, SW253, SW254, SW255: SW_SPDT, switches:8mm_push_button, symbol SW_SPDT
- added SW201, SW202, SW203, SW204, SW205, SW206, SW207, SW208, SW209, SW210, SW211, SW212, SW213, SW214, SW215, SW216, SW217, SW218, SW219, SW220, SW221, SW222, SW223, SW224, SW225, SW226, SW227, SW228, SW229, SW230, SW231, SW232, SW233, SW234, SW235, SW236, SW237, SW238, SW239, SW240, SW241, SW242, SW243, SW244, SW245, SW246, SW247, SW248, SW249, SW250, SW251, SW252, SW253, SW254, SW255: SW_SPDT_6pin, switches:8mm_push_button, symbol SW_SPDT_6pin
Connections:
- net DD11: now also SW225.1 (A)
- net DD12: now also SW226.1 (A)
- net DD13: now also SW227.1 (A)
- net DD14: now also SW228.1 (A)
- net DD15: now also SW229.1 (A)
- net DD16: now also SW230.1 (A)
- net DD17: now also SW231.1 (A)
- net DD18: now also SW232.1 (A)
- net DD21: now also SW233.1 (A)
- net DD22: now also SW234.1 (A)
- net DD23: now also SW235.1 (A)
- net DD24: now also SW236.1 (A)
- net DD25: now also SW237.1 (A)
- net DD26: now also SW238.1 (A)
- net DD27: now also SW239.1 (A)
- net DD28: now also SW240.1 (A)
- net GND: now also SW201.2 (B), SW201.4 (GND), SW201.5 (GND), SW201.6 (GND), SW202.2 (B), SW202.4 (GND), SW202.5 (GND), SW202.6 (GND), SW203.2 (B), SW203.4 (GND), SW203.5 (GND), SW203.6 (GND), SW204.2 (B), SW204.4 (GND), SW204.5 (GND), SW204.6 (GND), SW205.2 (B), SW205.4 (GND), SW205.5 (GND), SW205.6 (GND), SW206.2 (B), SW206.4 (GND), SW206.5 (GND), SW206.6 (GND), SW207.2 (B), SW207.4 (GND), SW207.5 (GND), SW207.6 (GND), SW208.2 (B), SW208.4 (GND), SW208.5 (GND), SW208.6 (GND), SW209.2 (B), SW209.4 (GND), SW209.5 (GND), SW209.6 (GND), SW210.2 (B), SW210.4 (GND), SW210.5 (GND), SW210.6 (GND), SW211.2 (B), SW211.4 (GND), SW211.5 (GND), SW211.6 (GND), SW212.2 (B), SW212.4 (GND), SW212.5 (GND), SW212.6 (GND), SW213.2 (B), SW213.4 (GND), SW213.5 (GND), SW213.6 (GND), SW214.2 (B), SW214.4 (GND), SW214.5 (GND), SW214.6 (GND), SW215.2 (B), SW215.4 (GND), SW215.5 (GND), SW215.6 (GND), SW216.2 (B), SW216.4 (GND), SW216.5 (GND), SW216.6 (GND), SW217.2 (B), SW217.4 (GND), SW217.5 (GND), SW217.6 (GND), SW218.2 (B), SW218.4 (GND), SW218.5 (GND), SW218.6 (GND), SW219.2 (B), SW219.4 (GND), SW219.5 (GND), SW219.6 (GND), SW220.2 (B), SW220.4 (GND), SW220.5 (GND), SW220.6 (GND), SW221.2 (B), SW221.4 (GND), SW221.5 (GND), SW221.6 (GND), SW222.2 (B), SW222.4 (GND), SW222.5 (GND), SW222.6 (GND), SW223.2 (B), SW223.4 (GND), SW223.5 (GND), SW223.6 (GND), SW224.2 (B), SW224.4 (GND), SW224.5 (GND), SW224.6 (GND), SW225.2 (B), SW225.4 (GND), SW225.5 (GND), SW225.6 (GND), SW226.2 (B), SW226.4 (GND), SW226.5 (GND), SW226.6 (GND), SW227.2 (B), SW227.4 (GND), SW227.5 (GND), SW227.6 (GND), SW228.2 (B), SW228.4 (GND), SW228.5 (GND), SW228.6 (GND), SW229.2 (B), SW229.4 (GND), SW229.5 (GND), SW229.6 (GND), SW230.2 (B), SW230.4 (GND), SW230.5 (GND), SW230.6 (GND), SW231.2 (B), SW231.4 (GND), SW231.5 (GND), SW231.6 (GND), SW232.2 (B), SW232.4 (GND), SW232.5 (GND), SW232.6 (GND), SW233.2 (B), SW233.4 (GND), SW233.5 (GND), SW233.6 (GND), SW234.2 (B), SW234.4 (GND), SW234.5 (GND), SW234.6 (GND), SW235.2 (B), SW235.4 (GND), SW235.5 (GND), SW235.6 (GND), SW236.2 (B), SW236.4 (GND), SW236.5 (GND), SW236.6 (GND), SW237.2 (B), SW237.4 (GND), SW237.5 (GND), SW237.6 (GND), SW238.2 (B), SW238.4 (GND), SW238.5 (GND), SW238.6 (GND), SW239.2 (B), SW239.4 (GND), SW239.5 (GND), SW239.6 (GND), SW240.2 (B), SW240.4 (GND), SW240.5 (GND), SW240.6 (GND), SW241.2 (B), SW241.4 (GND), SW241.5 (GND), SW241.6 (GND), SW242.2 (B), SW242.4 (GND), SW242.5 (GND), SW242.6 (GND), SW243.2 (B), SW243.4 (GND), SW243.5 (GND), SW243.6 (GND), SW244.2 (B), SW244.4 (GND), SW244.5 (GND), SW244.6 (GND), SW245.2 (B), SW245.4 (GND), SW245.5 (GND), SW245.6 (GND), SW246.2 (B), SW246.4 (GND), SW246.5 (GND), SW246.6 (GND), SW247.2 (B), SW247.4 (GND), SW247.5 (GND), SW247.6 (GND), SW248.2 (B), SW248.4 (GND), SW248.5 (GND), SW248.6 (GND), SW249.2 (B), SW249.4 (GND), SW249.5 (GND), SW249.6 (GND), SW250.2 (B), SW250.4 (GND), SW250.5 (GND), SW250.6 (GND), SW251.2 (B), SW251.4 (GND), SW251.5 (GND), SW251.6 (GND), SW252.2 (B), SW252.4 (GND), SW252.5 (GND), SW252.6 (GND), SW253.2 (B), SW253.4 (GND), SW253.5 (GND), SW253.6 (GND), SW254.2 (B), SW254.4 (GND), SW254.5 (GND), SW254.6 (GND), SW255.2 (B), SW255.4 (GND), SW255.5 (GND), SW255.6 (GND)
- net HD11: now also SW201.1 (A)
- net HD12: now also SW202.1 (A)
- net HD13: now also SW203.1 (A)
- net HD14: now also SW204.1 (A)
- net HD15: now also SW205.1 (A)
- net HD16: now also SW206.1 (A)
- net HD17: now also SW207.1 (A)
- net HD18: now also SW208.1 (A)
- net HD21: now also SW209.1 (A)
- net HD22: now also SW210.1 (A)
- net HD23: now also SW211.1 (A)
- net HD24: now also SW212.1 (A)
- net HD25: now also SW213.1 (A)
- net HD26: now also SW214.1 (A)
- net HD27: now also SW215.1 (A)
- net HD28: now also SW216.1 (A)
- net HD31: now also SW217.1 (A)
- net HD32: now also SW218.1 (A)
- net HD33: now also SW219.1 (A)
- net HD34: now also SW220.1 (A)
- net HD35: now also SW221.1 (A)
- net HD36: now also SW222.1 (A)
- net HD37: now also SW223.1 (A)
- net HD38: now also SW224.1 (A)
- net OD11: now also SW241.1 (A)
- net OD12: now also SW242.1 (A)
- net OD13: now also SW243.1 (A)
- net OD21: now also SW244.1 (A)
- net OD22: now also SW245.1 (A)
- net OD23: now also SW246.1 (A)
- net OD31: now also SW247.1 (A)
- net OD32: now also SW248.1 (A)
- net OD33: now also SW249.1 (A)
- net OD41: now also SW250.1 (A)
- net OD42: now also SW251.1 (A)
- net OD43: now also SW252.1 (A)
- net OD51: now also SW253.1 (A)
- net OD52: now also SW254.1 (A)
- net OD53: now also SW255.1 (A)
