File: Voicemeeter/file5AE700A4.sch (KiCad schematic (older format))
At the start: 15 parts, among them J501 CONN_01X05, J502 CONN_01X03, J503 CONN_01X05, J504 CONN_01X02, J505 CONN_01X03, J506 CONN_01X02, J507 DIN_5, J508 DIN_5, SW501 SW_Push, U501 stm32f103-china-MS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

Commit message: das
Connections:
- net M01 renamed M1
- net M02 renamed M2
- net M03 renamed M3
Changed lines of the file:
@@
 Connection ~ 7050 2100
-Wire Wire Line
-	4600 1900 3400 1900
-Wire Wire Line
-	4600 2100 3400 2100
-Wire Wire Line
-	4600 2300 3400 2300
 Wire Wire Line
 	4600 2500 3400 2500
@@
 	7850 3700 8000 3700
 Entry Wire Line
-	3300 2000 3400 1900
-Entry Wire Line
-	3300 2200 3400 2100
-Entry Wire Line
-	3300 2400 3400 2300
-Entry Wire Line
 	3300 2600 3400 2500
 Entry Wire Line
@@
 	3300 3800 3400 3700
 Wire Bus Line
-	3300 2000 3300 3800
+	3300 1700 3300 3800
 Wire Bus Line
-	3300 2000 3150 2000
-Text Label 3400 1900 0    60   ~ 0
-M01
-Text Label 3400 2100 0    60   ~ 0
-M02
-Text Label 3400 2300 0    60   ~ 0
-M03
+	3300 1700 3150 1700
 Text Label 7000 4100 0    60   ~ 0
 M11
@@
 Text HLabel 8000 3700 2    60   Input ~ 0
 M[1..27]
-Text HLabel 3150 2000 0    60   Input ~ 0
-M[01..27]
+Text HLabel 3150 1700 0    60   Input ~ 0
+M[1..27]
 NoConn ~ 9650 3550
 NoConn ~ 9500 3750
@@
 NoConn ~ 10700 2450
 Wire Wire Line
-	4600 5500 4150 5500
+	4150 5500 4600 5500
 Wire Wire Line
 	4400 5600 4400 5700
@@
 Text Label 3400 4300 0    60   ~ 0
 SK2
+Entry Wire Line
+	3300 2400 3400 2300
+Entry Wire Line
+	3300 2200 3400 2100
+Entry Wire Line
+	3300 2000 3400 1900
+Wire Wire Line
+	4600 1900 3400 1900
+Wire Wire Line
+	3400 2100 4600 2100
+Wire Wire Line
+	3400 2300 4600 2300
+Text Label 3400 1900 0    60   ~ 0
+M1
+Text Label 3400 2100 0    60   ~ 0
+M2
+Text Label 3400 2300 0    60   ~ 0
+M3
 $EndSCHEMATC

Commit message: rrr
asd
Parts:
- added C501, C502: 220uF, Capacitors_THT:CP_Radial_D6.3mm_P2.50mm, symbol CP
- added J509: Screw_Terminal_1x02, TerminalBlock:TerminalBlock_bornier-2_P5.08mm, symbol Screw_Terminal_1x02
Connections:
- net +3V3: now also C502.1
- net +5V: now also C501.1, J509.2
- net GND: now also C501.2, C502.2, J509.1
Other:
- moved on the sheet: J502
