File: Voicemeeter/test.kicad_pcb (KiCad board)
At the start: 2 copper layers, 344.9 x 217.8 mm, 193 parts, among them J501 CONN_01X05, J502 CONN_01X03, J503 CONN_01X05, J504 CONN_01X02, J505 CONN_01X03, J506 CONN_01X02, SW201 SW_SPDT, SW202 SW_SPDT, SW203 SW_SPDT, SW204 SW_SPDT, SW205 SW_SPDT, SW206 SW_SPDT, SW207 SW_SPDT, SW208 SW_SPDT, SW209 SW_SPDT, SW210 SW_SPDT, SW211 SW_SPDT, SW212 SW_SPDT, SW213 SW_SPDT, SW214 SW_SPDT, SW215 SW_SPDT, SW216 SW_SPDT, SW217 SW_SPDT, SW218 SW_SPDT, SW219 SW_SPDT, SW220 SW_SPDT, SW221 SW_SPDT, SW222 SW_SPDT, SW223 SW_SPDT, SW224 SW_SPDT, SW225 SW_SPDT, SW226 SW_SPDT, SW227 SW_SPDT, SW228 SW_SPDT, SW229 SW_SPDT, SW230 SW_SPDT, SW231 SW_SPDT, SW232 SW_SPDT, SW233 SW_SPDT, SW234 SW_SPDT, SW235 SW_SPDT, SW236 SW_SPDT, SW237 SW_SPDT, SW238 SW_SPDT, SW239 SW_SPDT, SW240 SW_SPDT, SW241 SW_SPDT, SW242 SW_SPDT, SW243 SW_SPDT, SW244 SW_SPDT, SW245 SW_SPDT, SW246 SW_SPDT, SW247 SW_SPDT, SW248 SW_SPDT, SW249 SW_SPDT, SW250 SW_SPDT, SW251 SW_SPDT, SW252 SW_SPDT, SW253 SW_SPDT, SW254 SW_SPDT, SW255 SW_SPDT, SW501 SW_Push, U401 74HC4051, U402 74HC4051, U403 74HC4051, U404 74HC4051, U405 74HC4051, U406 74HC4051, U407 74HC4051, U408 74HC4051, U409 74HC4051, U410 74HC4051, U501 stm32f103-china-MS, U502 PC817

Commit message: fsd
Parts:
- added LED617: SK9822, LEDs:LED_RGB_5050-6, F.Cu at (46.1, 232.1)
- added LED618: SK9822, LEDs:LED_RGB_5050-6, F.Cu at (66.9, 232.1)
- added LED619: SK9822, LEDs:LED_RGB_5050-6, F.Cu at (87.8, 232.1)
- added LED620: SK9822, LEDs:LED_RGB_5050-6, F.Cu at (108.6, 232.1)
- added LED621: SK9822, LEDs:LED_RGB_5050-6, F.Cu at (129.5, 232.1)
- added LED622: SK9822, LEDs:LED_RGB_5050-6, F.Cu at (150.3, 232.1)
- added LED623: SK9822, LEDs:LED_RGB_5050-6, F.Cu at (171.2, 232.1)
- added LED624: SK9822, LEDs:LED_RGB_5050-6, F.Cu at (192.0, 232.1)
- added LED625: SK9822, LEDs:LED_RGB_5050-6, F.Cu at (212.9, 232.1)
- added LED626: SK9822, LEDs:LED_RGB_5050-6, F.Cu at (233.7, 232.1)
- added LED627: SK9822, LEDs:LED_RGB_5050-6, F.Cu at (254.6, 232.1)
- added LED628: SK9822, LEDs:LED_RGB_5050-6, F.Cu at (275.4, 232.1)
- added LED629: SK9822, LEDs:LED_RGB_5050-6, F.Cu at (296.2, 232.1)
- added LED630: SK9822, LEDs:LED_RGB_5050-6, F.Cu at (317.1, 232.1)
- added LED631: SK9822, LEDs:LED_RGB_5050-6, F.Cu at (337.9, 232.1)
- added LED632: SK9822, LEDs:LED_RGB_5050-6, F.Cu at (358.8, 232.1)
- added REF**: via_single, myelin-kicad:via_single, F.Cu at (50.3, 212.1)
- added REF**: via_single, myelin-kicad:via_single, F.Cu at (91.9, 228.2)
- added REF**: via_single, myelin-kicad:via_single, F.Cu at (65.7, 169.4)
- added REF**: via_single, myelin-kicad:via_single, F.Cu at (46.2, 169.4)
- added REF**: via_single, myelin-kicad:via_single, F.Cu at (46.2, 168.3)
- added REF**: via_single, myelin-kicad:via_single, F.Cu at (65.7, 168.3)
- C302, C303, C305, C306, C308, C309, C311, C312, C315, C316: moved to F.Cu
- moved LED601 295.9 mm to (344.2, 118.9), turned to 180 degrees
- moved LED616 295.9 mm to (48.3, 118.9), turned to 180 degrees
- moved LED615 229.9 mm to (81.3, 118.9), turned to 180 degrees
- moved LED602 229.6 mm to (310.9, 118.9), turned to 180 degrees
- moved LED603 163.8 mm to (278.1, 118.9), turned to 180 degrees
- moved LED614 163.8 mm to (114.3, 118.9), turned to 180 degrees
- moved LED613 125.6 mm to (134.6, 58.4), turned to 90 degrees
- moved U403 115.4 mm to (103.1, 63.5), turned to 90 degrees
- moved LED604 111.7 mm to (245.4, 118.9), turned to 180 degrees
- moved U402 100.1 mm to (225.6, 146.8)
- moved LED605 86.3 mm to (212.3, 118.9), turned to 180 degrees
- moved LED612 85.8 mm to (134.6, 81.3), turned to 90 degrees
- moved SW501 80.8 mm to (215.1, 84.9)
- moved LED611 77.8 mm to (134.6, 104.1)
- moved LED606 77.6 mm to (197.4, 104.0)
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Connections:
- RV202 pad 1: +3V3 -> GND
- RV202 pad 3: GND -> +3V3
- RV203 pad 1: GND -> +3V3
- RV203 pad 3: +3V3 -> GND
- RV205 pad 1: +3V3 -> GND
- RV205 pad 3: GND -> +3V3
- RV206 pad 1: GND -> +3V3
- RV206 pad 3: +3V3 -> GND
- RV208 pad 1: +3V3 -> GND
- RV208 pad 3: GND -> +3V3
- RV209 pad 1: GND -> +3V3
- RV209 pad 3: +3V3 -> GND
- RV210 pad 1: +3V3 -> GND
- RV210 pad 3: GND -> +3V3
- RV212 pad 1: GND -> +3V3
- RV212 pad 3: +3V3 -> GND
- RV213 pad 1: GND -> +3V3
- RV213 pad 3: +3V3 -> GND
- RV214 pad 1: +3V3 -> GND
- RV214 pad 3: GND -> +3V3
- RV216 pad 1: GND -> +3V3
- RV216 pad 3: +3V3 -> GND
- RV217 pad 1: GND -> +3V3
- RV217 pad 3: +3V3 -> GND
- RV218 pad 1: +3V3 -> GND
- RV218 pad 3: GND -> +3V3
- RV219 pad 1: +3V3 -> GND
- RV219 pad 3: GND -> +3V3
- RV220 pad 1: +3V3 -> GND
- RV220 pad 3: GND -> +3V3
- RV221 pad 1: +3V3 -> GND
- RV221 pad 3: GND -> +3V3
- RV222 pad 1: +3V3 -> GND
- RV222 pad 3: GND -> +3V3
- U401 pad 1: /Mux/HA22 -> /Mux/HA13
- U401 pad 10: /Mux/M02 -> /Mux/M2
- U401 pad 11: /Mux/M01 -> /Mux/M1
- U401 pad 12: /Mux/HA21 -> /Mux/HA32
- U401 pad 13: /Mux/HA11 -> /Mux/HA31
- U401 pad 14: /Mux/HA12 -> /Mux/HA23
- U401 pad 15: /Mux/HA13 -> /Mux/HA11
- U401 pad 2: /Mux/HA31 -> /Mux/HA12
- U401 pad 4: /Mux/HA32 -> /Mux/HA21
- U401 pad 5: /Mux/HA23 -> /Mux/HA22
- U401 pad 9: /Mux/M03 -> /Mux/M3
- U402 pad 1: /Mux/OA4 -> Net-(U402-Pad1)
- U402 pad 10: /Mux/M02 -> /Mux/M2
- U402 pad 11: /Mux/M01 -> /Mux/M1
- U402 pad 12: /Mux/OA3 -> /Mux/OA2
- U402 pad 13: /Mux/HA33 -> /Mux/OA3
- U402 pad 14: /Mux/OA1 -> /Mux/OA4
- U402 pad 15: /Mux/OA2 -> /Mux/OA5
- U402 pad 2: Net-(U402-Pad2) -> /Mux/DA21
- U402 pad 4: Net-(U402-Pad4) -> /Mux/DA11
- U402 pad 5: /Mux/OA5 -> /Mux/OA1
- U402 pad 9: /Mux/M03 -> /Mux/M3
- U403 pad 1: /Mux/DA21 -> /Mux/DA23
- U403 pad 10: /Mux/M02 -> /Mux/M2
- U403 pad 11: /Mux/M01 -> /Mux/M1
- U403 pad 12: /Mux/DA14 -> /Mux/DA12
- U403 pad 13: /Mux/DA11 -> /Mux/DA13
- U403 pad 14: /Mux/DA12 -> /Mux/DA14
- U403 pad 15: /Mux/DA13 -> /Mux/DA22
- U403 pad 2: /Mux/DA23 -> /Mux/DA24
- U403 pad 4: /Mux/DA24 -> Net-(U403-Pad4)
- U403 pad 5: /Mux/DA22 -> /Mux/HA33
- U403 pad 9: /Mux/M03 -> /Mux/M3
- U404 pad 10: /Mux/M02 -> /Mux/M2
- U404 pad 11: /Mux/M01 -> /Mux/M1
- U404 pad 9: /Mux/M03 -> /Mux/M3
- U405 pad 10: /Mux/M02 -> /Mux/M2
- U405 pad 11: /Mux/M01 -> /Mux/M1
- U405 pad 9: /Mux/M03 -> /Mux/M3
- U406 pad 10: /Mux/M02 -> /Mux/M2
- U406 pad 11: /Mux/M01 -> /Mux/M1
- U406 pad 9: /Mux/M03 -> /Mux/M3
- U407 pad 10: /Mux/M02 -> /Mux/M2
- U407 pad 11: /Mux/M01 -> /Mux/M1
- U407 pad 9: /Mux/M03 -> /Mux/M3
- U408 pad 10: /Mux/M02 -> /Mux/M2
- U408 pad 11: /Mux/M01 -> /Mux/M1
- U408 pad 9: /Mux/M03 -> /Mux/M3
- U409 pad 10: /Mux/M02 -> /Mux/M2
- U409 pad 11: /Mux/M01 -> /Mux/M1
- U409 pad 9: /Mux/M03 -> /Mux/M3
- U410 pad 10: /Mux/M02 -> /Mux/M2
- U410 pad 11: /Mux/M01 -> /Mux/M1
- U410 pad 4: /Mux/OD52 -> /Mux/OD53
- U410 pad 5: /Mux/OD53 -> /Mux/OD52
- U410 pad 9: /Mux/M03 -> /Mux/M3
- U501 pad 1: /STM/M01 -> /Mux/M1
- U501 pad 2: /STM/M02 -> /Mux/M2
- U501 pad 3: /STM/M03 -> /Mux/M3
Routing:
- net +3V3: track 986.4 -> 69.1 mm
- net /Mux/M1: track 0.00 -> 594.9 mm, vias 0 -> 1
- net /Mux/M2: track 0.00 -> 591.4 mm, vias 0 -> 2
- net /Mux/M3: track 0.00 -> 585.5 mm, vias 0 -> 2
- net GND: track 452.2 -> 38.9 mm
- net /Mux/M21: track 0.00 -> 243.5 mm, vias 0 -> 5
- net /Mux/M01: track 210.3 -> 0.00 mm
- net /Mux/M02: track 210.1 -> 0.00 mm
- net /Mux/M03: track 206.4 -> 0.00 mm
- net /Mux/M22: track 0.00 -> 203.4 mm, vias 0 -> 4
- net /Mux/M23: track 0.00 -> 200.8 mm, vias 0 -> 3
- net /Mux/M11: track 0.00 -> 190.4 mm, vias 0 -> 2
- net /Mux/M24: track 0.00 -> 189.5 mm, vias 0 -> 4
- net /Mux/HA31: track 0.00 -> 183.1 mm, vias 0 -> 4
- net /Mux/M27: track 0.00 -> 162.0 mm, vias 0 -> 4
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- added copper zone on B.Cu, net +3V3
- added copper zone on F.Cu, net GND
Other:
- rule trace_min: 0.1524 -> 0.127
- rule via_min_drill: 0.2 -> 0.3
- rule via_min_size: 0.4 -> 0.6

Commit message: das
Parts:
- added REF**: via_single, myelin-kicad:via_single, F.Cu at (179.0, 124.0)
- added REF**: via_single, myelin-kicad:via_single, F.Cu at (271.1, 95.1)
- C313, C317: moved to F.Cu
- moved C311 25.5 mm to (164.3, 106.0), turned to 90 degrees
- moved C312 22.7 mm to (164.2, 83.2), turned to 90 degrees
- moved C316 16.0 mm to (194.7, 89.7), turned to 90 degrees
- moved C315 15.7 mm to (194.7, 96.3)
- moved C317 14.2 mm to (195.6, 48.9), turned to 270 degrees
- moved C313 8.79 mm to (164.7, 60.4)
- moved C310 1.97 mm to (148.6, 198.6)
- moved C314 1.78 mm to (180.6, 198.6)
Connections:
- SW201 pad 4: (no net) -> Net-(SW201-Pad4)
- SW201 pad 5: (no net) -> Net-(SW201-Pad5)
- SW201 pad 6: (no net) -> Net-(SW201-Pad6)
- SW202 pad 4: (no net) -> Net-(SW202-Pad4)
- SW202 pad 5: (no net) -> Net-(SW202-Pad5)
- SW202 pad 6: (no net) -> Net-(SW202-Pad6)
- SW203 pad 4: (no net) -> Net-(SW203-Pad4)
- SW203 pad 5: (no net) -> Net-(SW203-Pad5)
- SW203 pad 6: (no net) -> Net-(SW203-Pad6)
- SW204 pad 4: (no net) -> Net-(SW204-Pad4)
- SW204 pad 5: (no net) -> Net-(SW204-Pad5)
- SW204 pad 6: (no net) -> Net-(SW204-Pad6)
- SW205 pad 4: (no net) -> Net-(SW205-Pad4)
- SW205 pad 5: (no net) -> Net-(SW205-Pad5)
- SW205 pad 6: (no net) -> Net-(SW205-Pad6)
- SW206 pad 4: (no net) -> Net-(SW206-Pad4)
- SW206 pad 5: (no net) -> Net-(SW206-Pad5)
- SW206 pad 6: (no net) -> Net-(SW206-Pad6)
- SW207 pad 4: (no net) -> Net-(SW207-Pad4)
- SW207 pad 5: (no net) -> Net-(SW207-Pad5)
- SW207 pad 6: (no net) -> Net-(SW207-Pad6)
- SW208 pad 4: (no net) -> Net-(SW208-Pad4)
- SW208 pad 5: (no net) -> Net-(SW208-Pad5)
- SW208 pad 6: (no net) -> Net-(SW208-Pad6)
- SW209 pad 4: (no net) -> Net-(SW209-Pad4)
- SW209 pad 5: (no net) -> Net-(SW209-Pad5)
- SW209 pad 6: (no net) -> Net-(SW209-Pad6)
- SW210 pad 4: (no net) -> Net-(SW210-Pad4)
- SW210 pad 5: (no net) -> Net-(SW210-Pad5)
- SW210 pad 6: (no net) -> Net-(SW210-Pad6)
- SW211 pad 4: (no net) -> Net-(SW211-Pad4)
- SW211 pad 5: (no net) -> Net-(SW211-Pad5)
- SW211 pad 6: (no net) -> Net-(SW211-Pad6)
- SW212 pad 4: (no net) -> Net-(SW212-Pad4)
- SW212 pad 5: (no net) -> Net-(SW212-Pad5)
- SW212 pad 6: (no net) -> Net-(SW212-Pad6)
- SW213 pad 4: (no net) -> Net-(SW213-Pad4)
- SW213 pad 5: (no net) -> Net-(SW213-Pad5)
- SW213 pad 6: (no net) -> Net-(SW213-Pad6)
- SW214 pad 4: (no net) -> Net-(SW214-Pad4)
- SW214 pad 5: (no net) -> Net-(SW214-Pad5)
- SW214 pad 6: (no net) -> Net-(SW214-Pad6)
- SW215 pad 4: (no net) -> Net-(SW215-Pad4)
- SW215 pad 5: (no net) -> Net-(SW215-Pad5)
- SW215 pad 6: (no net) -> Net-(SW215-Pad6)
- SW216 pad 4: (no net) -> Net-(SW216-Pad4)
- SW216 pad 5: (no net) -> Net-(SW216-Pad5)
- SW216 pad 6: (no net) -> Net-(SW216-Pad6)
- SW217 pad 4: (no net) -> Net-(SW217-Pad4)
- SW217 pad 5: (no net) -> Net-(SW217-Pad5)
- SW217 pad 6: (no net) -> Net-(SW217-Pad6)
- SW218 pad 4: (no net) -> Net-(SW218-Pad4)
- SW218 pad 5: (no net) -> Net-(SW218-Pad5)
- SW218 pad 6: (no net) -> Net-(SW218-Pad6)
- SW219 pad 4: (no net) -> Net-(SW219-Pad4)
- SW219 pad 5: (no net) -> Net-(SW219-Pad5)
- SW219 pad 6: (no net) -> Net-(SW219-Pad6)
- SW220 pad 4: (no net) -> Net-(SW220-Pad4)
- SW220 pad 5: (no net) -> Net-(SW220-Pad5)
- SW220 pad 6: (no net) -> Net-(SW220-Pad6)
- SW221 pad 4: (no net) -> Net-(SW221-Pad4)
- SW221 pad 5: (no net) -> Net-(SW221-Pad5)
- SW221 pad 6: (no net) -> Net-(SW221-Pad6)
- SW222 pad 4: (no net) -> Net-(SW222-Pad4)
- SW222 pad 5: (no net) -> Net-(SW222-Pad5)
- SW222 pad 6: (no net) -> Net-(SW222-Pad6)
- SW223 pad 4: (no net) -> Net-(SW223-Pad4)
- SW223 pad 5: (no net) -> Net-(SW223-Pad5)
- SW223 pad 6: (no net) -> Net-(SW223-Pad6)
- SW224 pad 4: (no net) -> Net-(SW224-Pad4)
- SW224 pad 5: (no net) -> Net-(SW224-Pad5)
- SW224 pad 6: (no net) -> Net-(SW224-Pad6)
- SW225 pad 4: (no net) -> Net-(SW225-Pad4)
- SW225 pad 5: (no net) -> Net-(SW225-Pad5)
- SW225 pad 6: (no net) -> Net-(SW225-Pad6)
- SW226 pad 4: (no net) -> Net-(SW226-Pad4)
- SW226 pad 5: (no net) -> Net-(SW226-Pad5)
- SW226 pad 6: (no net) -> Net-(SW226-Pad6)
- SW227 pad 4: (no net) -> Net-(SW227-Pad4)
- SW227 pad 5: (no net) -> Net-(SW227-Pad5)
- SW227 pad 6: (no net) -> Net-(SW227-Pad6)
- SW228 pad 4: (no net) -> Net-(SW228-Pad4)
- SW228 pad 5: (no net) -> Net-(SW228-Pad5)
- SW228 pad 6: (no net) -> Net-(SW228-Pad6)
- SW229 pad 4: (no net) -> Net-(SW229-Pad4)
- SW229 pad 5: (no net) -> Net-(SW229-Pad5)
- SW229 pad 6: (no net) -> Net-(SW229-Pad6)
- SW230 pad 4: (no net) -> Net-(SW230-Pad4)
- SW230 pad 5: (no net) -> Net-(SW230-Pad5)
- SW230 pad 6: (no net) -> Net-(SW230-Pad6)
- SW231 pad 4: (no net) -> Net-(SW231-Pad4)
- SW231 pad 5: (no net) -> Net-(SW231-Pad5)
- SW231 pad 6: (no net) -> Net-(SW231-Pad6)
- SW232 pad 4: (no net) -> Net-(SW232-Pad4)
- SW232 pad 5: (no net) -> Net-(SW232-Pad5)
- SW232 pad 6: (no net) -> Net-(SW232-Pad6)
- SW233 pad 4: (no net) -> Net-(SW233-Pad4)
- SW233 pad 5: (no net) -> Net-(SW233-Pad5)
- SW233 pad 6: (no net) -> Net-(SW233-Pad6)
- SW234 pad 4: (no net) -> Net-(SW234-Pad4)
- SW234 pad 5: (no net) -> Net-(SW234-Pad5)
- SW234 pad 6: (no net) -> Net-(SW234-Pad6)
- SW235 pad 4: (no net) -> Net-(SW235-Pad4)
- SW235 pad 5: (no net) -> Net-(SW235-Pad5)
- SW235 pad 6: (no net) -> Net-(SW235-Pad6)
- SW236 pad 4: (no net) -> Net-(SW236-Pad4)
- SW236 pad 5: (no net) -> Net-(SW236-Pad5)
- SW236 pad 6: (no net) -> Net-(SW236-Pad6)
- SW237 pad 4: (no net) -> Net-(SW237-Pad4)
- SW237 pad 5: (no net) -> Net-(SW237-Pad5)
- SW237 pad 6: (no net) -> Net-(SW237-Pad6)
- SW238 pad 4: (no net) -> Net-(SW238-Pad4)
- SW238 pad 5: (no net) -> Net-(SW238-Pad5)
- SW238 pad 6: (no net) -> Net-(SW238-Pad6)
- SW239 pad 4: (no net) -> Net-(SW239-Pad4)
- SW239 pad 5: (no net) -> Net-(SW239-Pad5)
- SW239 pad 6: (no net) -> Net-(SW239-Pad6)
- SW240 pad 4: (no net) -> Net-(SW240-Pad4)
- SW240 pad 5: (no net) -> Net-(SW240-Pad5)
- SW240 pad 6: (no net) -> Net-(SW240-Pad6)
- SW241 pad 4: (no net) -> Net-(SW241-Pad4)
- SW241 pad 5: (no net) -> Net-(SW241-Pad5)
- SW241 pad 6: (no net) -> Net-(SW241-Pad6)
- SW242 pad 4: (no net) -> Net-(SW242-Pad4)
- SW242 pad 5: (no net) -> Net-(SW242-Pad5)
- SW242 pad 6: (no net) -> Net-(SW242-Pad6)
- SW243 pad 4: (no net) -> Net-(SW243-Pad4)
- SW243 pad 5: (no net) -> Net-(SW243-Pad5)
- SW243 pad 6: (no net) -> Net-(SW243-Pad6)
- SW244 pad 4: (no net) -> Net-(SW244-Pad4)
- SW244 pad 5: (no net) -> Net-(SW244-Pad5)
- SW244 pad 6: (no net) -> Net-(SW244-Pad6)
- SW245 pad 4: (no net) -> Net-(SW245-Pad4)
- SW245 pad 5: (no net) -> Net-(SW245-Pad5)
- SW245 pad 6: (no net) -> Net-(SW245-Pad6)
- SW246 pad 4: (no net) -> Net-(SW246-Pad4)
- SW246 pad 5: (no net) -> Net-(SW246-Pad5)
- SW246 pad 6: (no net) -> Net-(SW246-Pad6)
- SW247 pad 4: (no net) -> Net-(SW247-Pad4)
- SW247 pad 5: (no net) -> Net-(SW247-Pad5)
- SW247 pad 6: (no net) -> Net-(SW247-Pad6)
- SW248 pad 4: (no net) -> Net-(SW248-Pad4)
- SW248 pad 5: (no net) -> Net-(SW248-Pad5)
- SW248 pad 6: (no net) -> Net-(SW248-Pad6)
- SW249 pad 4: (no net) -> Net-(SW249-Pad4)
- SW249 pad 5: (no net) -> Net-(SW249-Pad5)
- SW249 pad 6: (no net) -> Net-(SW249-Pad6)
- SW250 pad 4: (no net) -> Net-(SW250-Pad4)
- SW250 pad 5: (no net) -> Net-(SW250-Pad5)
- SW250 pad 6: (no net) -> Net-(SW250-Pad6)
- SW251 pad 4: (no net) -> Net-(SW251-Pad4)
- SW251 pad 5: (no net) -> Net-(SW251-Pad5)
- SW251 pad 6: (no net) -> Net-(SW251-Pad6)
- SW252 pad 4: (no net) -> Net-(SW252-Pad4)
- SW252 pad 5: (no net) -> Net-(SW252-Pad5)
- SW252 pad 6: (no net) -> Net-(SW252-Pad6)
- SW253 pad 4: (no net) -> Net-(SW253-Pad4)
- SW253 pad 5: (no net) -> Net-(SW253-Pad5)
- SW253 pad 6: (no net) -> Net-(SW253-Pad6)
- SW254 pad 4: (no net) -> Net-(SW254-Pad4)
- SW254 pad 5: (no net) -> Net-(SW254-Pad5)
- SW254 pad 6: (no net) -> Net-(SW254-Pad6)
- SW255 pad 4: (no net) -> Net-(SW255-Pad4)
- SW255 pad 5: (no net) -> Net-(SW255-Pad5)
- SW255 pad 6: (no net) -> Net-(SW255-Pad6)
Routing:
- net +5V: track 7.62 -> 298.8 mm, vias 0 -> 10
- net /Mux/DD21: track 3.20 -> 128.4 mm, vias 0 -> 1
- net /Mux/DD11: track 3.29 -> 127.5 mm, vias 0 -> 2
- net /Mux/DA24: track 0.00 -> 123.7 mm, vias 0 -> 1
- net /Mux/DA22: track 0.00 -> 123.1 mm, vias 0 -> 2
- net /Mux/DD22: track 3.20 -> 111.4 mm
- net /Mux/DD12: track 3.23 -> 109.8 mm, vias 0 -> 3
- net /Mux/DA23: track 0.00 -> 106.3 mm, vias 0 -> 3
- net Net-(LED608-Pad6): track 0.00 -> 95.3 mm, vias 0 -> 6
- net Net-(LED608-Pad5): track 0.00 -> 94.4 mm, vias 0 -> 6
- net /Mux/DD13: track 3.23 -> 94.9 mm
- net /Mux/DD23: track 3.20 -> 91.6 mm
- net /Mux/DA12: track 0.00 -> 80.3 mm, vias 0 -> 2
- net /Mux/HA32: track 3.18 -> 77.1 mm, vias 0 -> 3
- net /Mux/M3: track 585.5 -> 659.2 mm, vias 2 -> 3
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
Commit message: asf
Parts:
- added REF**: via_single, myelin-kicad:via_single, F.Cu at (100.3, 99.6)
- added REF**: via_single, myelin-kicad:via_single, F.Cu at (100.3, 92.5)
- added REF**: via_single, myelin-kicad:via_single, F.Cu at (99.6, 99.6)
- added REF**: via_single, myelin-kicad:via_single, F.Cu at (98.8, 99.6)
- added REF**: via_single, myelin-kicad:via_single, F.Cu at (98.8, 92.5)
- added REF**: via_single, myelin-kicad:via_single, F.Cu at (99.6, 92.5)
- SW201, SW202, SW203, SW204, SW205, SW206, SW207, SW208, SW209, SW210, SW211, SW212, SW213, SW214, SW215, SW216, SW217, SW218, SW219, SW220, SW221, SW222, SW223, SW224, SW225, SW226, SW227, SW228, SW229, SW230, SW231, SW232, SW233, SW234, SW235, SW236, SW237, SW238, SW239, SW240, SW241, SW242, SW243, SW244, SW245, SW246, SW247, SW248, SW249, SW250, SW251, SW252, SW253, SW254, SW255: value SW_SPDT -> SW_SPDT_6pin
Connections:
- SW201 pad 4: Net-(SW201-Pad4) -> GND
- SW201 pad 5: Net-(SW201-Pad5) -> GND
- SW201 pad 6: Net-(SW201-Pad6) -> GND
- SW202 pad 4: Net-(SW202-Pad4) -> GND
- SW202 pad 5: Net-(SW202-Pad5) -> GND
- SW202 pad 6: Net-(SW202-Pad6) -> GND
- SW203 pad 4: Net-(SW203-Pad4) -> GND
- SW203 pad 5: Net-(SW203-Pad5) -> GND
- SW203 pad 6: Net-(SW203-Pad6) -> GND
- SW204 pad 4: Net-(SW204-Pad4) -> GND
- SW204 pad 5: Net-(SW204-Pad5) -> GND
- SW204 pad 6: Net-(SW204-Pad6) -> GND
- SW205 pad 4: Net-(SW205-Pad4) -> GND
- SW205 pad 5: Net-(SW205-Pad5) -> GND
- SW205 pad 6: Net-(SW205-Pad6) -> GND
- SW206 pad 4: Net-(SW206-Pad4) -> GND
- SW206 pad 5: Net-(SW206-Pad5) -> GND
- SW206 pad 6: Net-(SW206-Pad6) -> GND
- SW207 pad 4: Net-(SW207-Pad4) -> GND
- SW207 pad 5: Net-(SW207-Pad5) -> GND
- SW207 pad 6: Net-(SW207-Pad6) -> GND
- SW208 pad 4: Net-(SW208-Pad4) -> GND
- SW208 pad 5: Net-(SW208-Pad5) -> GND
- SW208 pad 6: Net-(SW208-Pad6) -> GND
- SW209 pad 4: Net-(SW209-Pad4) -> GND
- SW209 pad 5: Net-(SW209-Pad5) -> GND
- SW209 pad 6: Net-(SW209-Pad6) -> GND
- SW210 pad 4: Net-(SW210-Pad4) -> GND
- SW210 pad 5: Net-(SW210-Pad5) -> GND
- SW210 pad 6: Net-(SW210-Pad6) -> GND
- SW211 pad 4: Net-(SW211-Pad4) -> GND
- SW211 pad 5: Net-(SW211-Pad5) -> GND
- SW211 pad 6: Net-(SW211-Pad6) -> GND
- SW212 pad 4: Net-(SW212-Pad4) -> GND
- SW212 pad 5: Net-(SW212-Pad5) -> GND
- SW212 pad 6: Net-(SW212-Pad6) -> GND
- SW213 pad 4: Net-(SW213-Pad4) -> GND
- SW213 pad 5: Net-(SW213-Pad5) -> GND
- SW213 pad 6: Net-(SW213-Pad6) -> GND
- SW214 pad 4: Net-(SW214-Pad4) -> GND
- SW214 pad 5: Net-(SW214-Pad5) -> GND
- SW214 pad 6: Net-(SW214-Pad6) -> GND
- SW215 pad 4: Net-(SW215-Pad4) -> GND
- SW215 pad 5: Net-(SW215-Pad5) -> GND
- SW215 pad 6: Net-(SW215-Pad6) -> GND
- SW216 pad 4: Net-(SW216-Pad4) -> GND
- SW216 pad 5: Net-(SW216-Pad5) -> GND
- SW216 pad 6: Net-(SW216-Pad6) -> GND
- SW217 pad 4: Net-(SW217-Pad4) -> GND
- SW217 pad 5: Net-(SW217-Pad5) -> GND
- SW217 pad 6: Net-(SW217-Pad6) -> GND
- SW218 pad 4: Net-(SW218-Pad4) -> GND
- SW218 pad 5: Net-(SW218-Pad5) -> GND
- SW218 pad 6: Net-(SW218-Pad6) -> GND
- SW219 pad 4: Net-(SW219-Pad4) -> GND
- SW219 pad 5: Net-(SW219-Pad5) -> GND
- SW219 pad 6: Net-(SW219-Pad6) -> GND
- SW220 pad 4: Net-(SW220-Pad4) -> GND
- SW220 pad 5: Net-(SW220-Pad5) -> GND
- SW220 pad 6: Net-(SW220-Pad6) -> GND
- SW221 pad 4: Net-(SW221-Pad4) -> GND
- SW221 pad 5: Net-(SW221-Pad5) -> GND
- SW221 pad 6: Net-(SW221-Pad6) -> GND
- SW222 pad 4: Net-(SW222-Pad4) -> GND
- SW222 pad 5: Net-(SW222-Pad5) -> GND
- SW222 pad 6: Net-(SW222-Pad6) -> GND
- SW223 pad 4: Net-(SW223-Pad4) -> GND
- SW223 pad 5: Net-(SW223-Pad5) -> GND
- SW223 pad 6: Net-(SW223-Pad6) -> GND
- SW224 pad 4: Net-(SW224-Pad4) -> GND
- SW224 pad 5: Net-(SW224-Pad5) -> GND
- SW224 pad 6: Net-(SW224-Pad6) -> GND
- SW225 pad 4: Net-(SW225-Pad4) -> GND
- SW225 pad 5: Net-(SW225-Pad5) -> GND
- SW225 pad 6: Net-(SW225-Pad6) -> GND
- SW226 pad 4: Net-(SW226-Pad4) -> GND
- SW226 pad 5: Net-(SW226-Pad5) -> GND
- SW226 pad 6: Net-(SW226-Pad6) -> GND
- SW227 pad 4: Net-(SW227-Pad4) -> GND
- SW227 pad 5: Net-(SW227-Pad5) -> GND
- SW227 pad 6: Net-(SW227-Pad6) -> GND
- SW228 pad 4: Net-(SW228-Pad4) -> GND
- SW228 pad 5: Net-(SW228-Pad5) -> GND
- SW228 pad 6: Net-(SW228-Pad6) -> GND
- SW229 pad 4: Net-(SW229-Pad4) -> GND
- SW229 pad 5: Net-(SW229-Pad5) -> GND
- SW229 pad 6: Net-(SW229-Pad6) -> GND
- SW230 pad 4: Net-(SW230-Pad4) -> GND
- SW230 pad 5: Net-(SW230-Pad5) -> GND
- SW230 pad 6: Net-(SW230-Pad6) -> GND
- SW231 pad 4: Net-(SW231-Pad4) -> GND
- SW231 pad 5: Net-(SW231-Pad5) -> GND
- SW231 pad 6: Net-(SW231-Pad6) -> GND
- SW232 pad 4: Net-(SW232-Pad4) -> GND
- SW232 pad 5: Net-(SW232-Pad5) -> GND
- SW232 pad 6: Net-(SW232-Pad6) -> GND
- SW233 pad 4: Net-(SW233-Pad4) -> GND
- SW233 pad 5: Net-(SW233-Pad5) -> GND
- SW233 pad 6: Net-(SW233-Pad6) -> GND
- SW234 pad 4: Net-(SW234-Pad4) -> GND
- SW234 pad 5: Net-(SW234-Pad5) -> GND
- SW234 pad 6: Net-(SW234-Pad6) -> GND
- SW235 pad 4: Net-(SW235-Pad4) -> GND
- SW235 pad 5: Net-(SW235-Pad5) -> GND
- SW235 pad 6: Net-(SW235-Pad6) -> GND
- SW236 pad 4: Net-(SW236-Pad4) -> GND
- SW236 pad 5: Net-(SW236-Pad5) -> GND
- SW236 pad 6: Net-(SW236-Pad6) -> GND
- SW237 pad 4: Net-(SW237-Pad4) -> GND
- SW237 pad 5: Net-(SW237-Pad5) -> GND
- SW237 pad 6: Net-(SW237-Pad6) -> GND
- SW238 pad 4: Net-(SW238-Pad4) -> GND
- SW238 pad 5: Net-(SW238-Pad5) -> GND
- SW238 pad 6: Net-(SW238-Pad6) -> GND
- SW239 pad 4: Net-(SW239-Pad4) -> GND
- SW239 pad 5: Net-(SW239-Pad5) -> GND
- SW239 pad 6: Net-(SW239-Pad6) -> GND
- SW240 pad 4: Net-(SW240-Pad4) -> GND
- SW240 pad 5: Net-(SW240-Pad5) -> GND
- SW240 pad 6: Net-(SW240-Pad6) -> GND
- SW241 pad 4: Net-(SW241-Pad4) -> GND
- SW241 pad 5: Net-(SW241-Pad5) -> GND
- SW241 pad 6: Net-(SW241-Pad6) -> GND
- SW242 pad 4: Net-(SW242-Pad4) -> GND
- SW242 pad 5: Net-(SW242-Pad5) -> GND
- SW242 pad 6: Net-(SW242-Pad6) -> GND
- SW243 pad 4: Net-(SW243-Pad4) -> GND
- SW243 pad 5: Net-(SW243-Pad5) -> GND
- SW243 pad 6: Net-(SW243-Pad6) -> GND
- SW244 pad 4: Net-(SW244-Pad4) -> GND
- SW244 pad 5: Net-(SW244-Pad5) -> GND
- SW244 pad 6: Net-(SW244-Pad6) -> GND
- SW245 pad 4: Net-(SW245-Pad4) -> GND
- SW245 pad 5: Net-(SW245-Pad5) -> GND
- SW245 pad 6: Net-(SW245-Pad6) -> GND
- SW246 pad 4: Net-(SW246-Pad4) -> GND
- SW246 pad 5: Net-(SW246-Pad5) -> GND
- SW246 pad 6: Net-(SW246-Pad6) -> GND
- SW247 pad 4: Net-(SW247-Pad4) -> GND
- SW247 pad 5: Net-(SW247-Pad5) -> GND
- SW247 pad 6: Net-(SW247-Pad6) -> GND
- SW248 pad 4: Net-(SW248-Pad4) -> GND
- SW248 pad 5: Net-(SW248-Pad5) -> GND
- SW248 pad 6: Net-(SW248-Pad6) -> GND
- SW249 pad 4: Net-(SW249-Pad4) -> GND
- SW249 pad 5: Net-(SW249-Pad5) -> GND
- SW249 pad 6: Net-(SW249-Pad6) -> GND
- SW250 pad 4: Net-(SW250-Pad4) -> GND
- SW250 pad 5: Net-(SW250-Pad5) -> GND
- SW250 pad 6: Net-(SW250-Pad6) -> GND
- SW251 pad 4: Net-(SW251-Pad4) -> GND
- SW251 pad 5: Net-(SW251-Pad5) -> GND
- SW251 pad 6: Net-(SW251-Pad6) -> GND
- SW252 pad 4: Net-(SW252-Pad4) -> GND
- SW252 pad 5: Net-(SW252-Pad5) -> GND
- SW252 pad 6: Net-(SW252-Pad6) -> GND
- SW253 pad 4: Net-(SW253-Pad4) -> GND
- SW253 pad 5: Net-(SW253-Pad5) -> GND
- SW253 pad 6: Net-(SW253-Pad6) -> GND
- SW254 pad 4: Net-(SW254-Pad4) -> GND
- SW254 pad 5: Net-(SW254-Pad5) -> GND
- SW254 pad 6: Net-(SW254-Pad6) -> GND
- SW255 pad 4: Net-(SW255-Pad4) -> GND
- SW255 pad 5: Net-(SW255-Pad5) -> GND
- SW255 pad 6: Net-(SW255-Pad6) -> GND
Routing:
- net +5V: track 298.8 -> 1072.1 mm, vias 10 -> 27
- net Net-(LED616-Pad5): track 0.00 -> 120.8 mm, vias 0 -> 2
- net Net-(LED616-Pad6): track 0.00 -> 113.5 mm, vias 0 -> 2
- net Net-(LED613-Pad5): track 0.00 -> 76.1 mm, vias 0 -> 2
- net Net-(LED613-Pad6): track 0.00 -> 72.7 mm, vias 0 -> 2
- net Net-(LED615-Pad6): track 0.00 -> 30.6 mm
- net Net-(LED615-Pad5): track 0.00 -> 30.2 mm
- net Net-(LED614-Pad6): track 0.00 -> 30.0 mm
- net Net-(LED614-Pad5): track 0.00 -> 29.7 mm
- net Net-(SW501-Pad2): track 0.00 -> 27.6 mm
- net +3V3: track 73.7 -> 95.6 mm
- net Net-(LED610-Pad6): track 0.00 -> 20.2 mm
- net Net-(LED612-Pad6): track 0.00 -> 18.1 mm
- net Net-(LED612-Pad5): track 0.00 -> 18.1 mm
- net Net-(LED611-Pad6): track 0.00 -> 18.1 mm
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
Commit message: rrr
asd
Parts:
- added C501: 220uF, Capacitors_THT:CP_Radial_D6.3mm_P2.50mm, F.Cu at (282.2, 108.2)
- added C502: 220uF, Capacitors_THT:CP_Radial_D6.3mm_P2.50mm, F.Cu at (241.0, 57.1)
- added J509: Screw_Terminal_1x02, TerminalBlock:TerminalBlock_bornier-2_P5.08mm, F.Cu at (293.4, 108.2)
- moved SW501 0.08 mm to (215.2, 84.9)
Routing:
- net +5V: track 1072.1 -> 1164.6 mm
- net Net-(SW501-Pad2): track 27.6 -> 26.6 mm
Other:
- board size 344.9 x 217.8 mm -> 348.5 x 271.7 mm
